Commit message: 升降导程修复,上下位机通信修复

File: src/joint_hardware/description/lift.ros2_control.xacro (robot description, xacro)
@@ -7,5 +7,5 @@
             ethercat_interface:=enp5s0 dc_assign_activate:=0 dc_sync0_shift_ns:=0
             command_units_per_rev:=10000 encoder_counts_per_rev:=131072
-            lead_mm_per_rev:=10.0 lift_sign:=-1.0 position_min_m:=-1.0
+            lead_mm_per_rev:=3.333333333 lift_sign:=-1.0 position_min_m:=-1.0
             position_max_m:=0.0 max_rpm:=360 brake_control_enabled:=false
             position_limit_recovery_max_rpm:=300
@@ -44,4 +44,5 @@
         <param name="position_min_m">${position_min_m}</param>
         <param name="position_max_m">${position_max_m}</param>
+        <param name="reset_max_search_travel_m">${lift_cfg['reset_max_search_travel_m']}</param>
         <param name="max_rpm">${max_rpm}</param>
         <param name="position_limit_recovery_max_rpm">${position_limit_recovery_max_rpm}</param>

File: src/joint_hardware/description/lift_test.urdf.xacro (robot description, xacro)
@@ -15,5 +15,5 @@
   <xacro:arg name="command_units_per_rev" default="10000"/>
   <xacro:arg name="encoder_counts_per_rev" default="131072"/>
-  <xacro:arg name="lead_mm_per_rev" default="10.0"/>
+  <xacro:arg name="lead_mm_per_rev" default="3.333333333"/>
   <xacro:arg name="lift_sign" default="-1.0"/>
   <xacro:arg name="position_min_m" default="-1.0"/>
@@ -79,5 +79,5 @@
     <child link="lift_carriage"/>
     <axis xyz="0 0 1"/>
-    <limit lower="-1.0" upper="0.0" velocity="0.060" effort="1000.0"/>
+    <limit lower="-1.0" upper="0.0" velocity="0.020" effort="1000.0"/>
   </joint>
 </robot>

Commit message: 验证搬箱子workflow可运行，完善tools脚本，基于TCP协议

File: src/joint_hardware/description/lift.ros2_control.xacro (robot description, xacro)
@@ -8,5 +8,5 @@
             command_units_per_rev:=10000 encoder_counts_per_rev:=131072
             lead_mm_per_rev:=3.333333333 lift_sign:=-1.0 position_min_m:=-1.0
-            position_max_m:=0.0 max_rpm:=360 brake_control_enabled:=false
+            position_max_m:=0.0 max_rpm:=1440 brake_control_enabled:=false
             position_limit_recovery_max_rpm:=300
             limit_switch_enabled:=false limit_switch_positive_bit:=-1

File: src/joint_hardware/description/lift_test.urdf.xacro (robot description, xacro)
@@ -19,5 +19,5 @@
   <xacro:arg name="position_min_m" default="-1.0"/>
   <xacro:arg name="position_max_m" default="0.0"/>
-  <xacro:arg name="max_rpm" default="360"/>
+  <xacro:arg name="max_rpm" default="1440"/>
   <xacro:arg name="position_limit_recovery_max_rpm" default="300"/>
   <xacro:arg name="brake_control_enabled" default="false"/>
@@ -79,5 +79,5 @@
     <child link="lift_carriage"/>
     <axis xyz="0 0 1"/>
-    <limit lower="-1.0" upper="0.0" velocity="0.020" effort="1000.0"/>
+    <limit lower="-1.0" upper="0.0" velocity="0.080" effort="1000.0"/>
   </joint>
 </robot>

Commit message: nothing

File: src/joint_hardware/description/lift.ros2_control.xacro (robot description, xacro)
@@ -38,13 +38,13 @@
         <param name="dc_sync0_shift_ns">${dc_sync0_shift_ns}</param>
         <param name="motor_id">LVM08008H3G3-M17</param>
-        <param name="lead_mm_per_rev">${lead_mm_per_rev}</param>
-        <param name="lift_sign">${lift_sign}</param>
+        <param name="lead_mm_per_rev">${lift_cfg['lead_mm_per_rev']}</param>
+        <param name="lift_sign">${lift_cfg['lift_sign']}</param>
         <param name="command_units_per_rev">${command_units_per_rev}</param>
         <param name="encoder_counts_per_rev">${encoder_counts_per_rev}</param>
-        <param name="position_min_m">${position_min_m}</param>
-        <param name="position_max_m">${position_max_m}</param>
+        <param name="position_min_m">${lift_cfg['position_min_m']}</param>
+        <param name="position_max_m">${lift_cfg['position_max_m']}</param>
         <param name="reset_max_search_travel_m">${lift_cfg['reset_max_search_travel_m']}</param>
-        <param name="max_rpm">${max_rpm}</param>
-        <param name="position_limit_recovery_max_rpm">${position_limit_recovery_max_rpm}</param>
+        <param name="max_rpm">${lift_cfg['max_rpm']}</param>
+        <param name="position_limit_recovery_max_rpm">${lift_cfg['position_limit_recovery_max_rpm']}</param>
         <param name="brake_control_enabled">${brake_control_enabled}</param>
         <param name="limit_switch_enabled">${limit_switch_enabled}</param>

File: src/joint_hardware/description/lift_test.urdf.xacro (robot description, xacro)
@@ -36,4 +36,5 @@
   <xacro:arg name="use_persistent_zero_offset" default="false"/>
   <xacro:arg name="zero_offset_file" default="/tmp/joint_hardware_lift_zero_offset.cfg"/>
+  <xacro:property name="lift_cfg" value="${xacro.load_yaml('$(arg hardware_config_file)')}"/>
   <xacro:include filename="$(find joint_hardware)/description/lift.ros2_control.xacro"/>
   <xacro:joint_lift_ros2_control
@@ -79,5 +80,9 @@
     <child link="lift_carriage"/>
     <axis xyz="0 0 1"/>
-    <limit lower="-1.0" upper="0.0" velocity="0.080" effort="1000.0"/>
+    <limit
+      lower="${lift_cfg['position_min_m']}"
+      upper="${lift_cfg['position_max_m']}"
+      velocity="${lift_cfg['max_feedback_velocity_mps']}"
+      effort="1000.0"/>
   </joint>
 </robot>

Commit message: nothing

File: src/joint_hardware/description/lift.ros2_control.xacro (robot description, xacro)
@@ -7,6 +7,6 @@
             ethercat_interface:=enp5s0 dc_assign_activate:=0 dc_sync0_shift_ns:=0
             command_units_per_rev:=10000 encoder_counts_per_rev:=131072
-            lead_mm_per_rev:=10.0 lift_sign:=-1.0 position_min_m:=-1.0
-            position_max_m:=0.0 max_rpm:=360 brake_control_enabled:=false
+            lead_mm_per_rev:=3.333333333 lift_sign:=-1.0 position_min_m:=-1.0
+            position_max_m:=0.0 max_rpm:=1440 brake_control_enabled:=false
             position_limit_recovery_max_rpm:=300
             limit_switch_enabled:=false limit_switch_positive_bit:=-1
@@ -38,12 +38,13 @@
         <param name="dc_sync0_shift_ns">${dc_sync0_shift_ns}</param>
         <param name="motor_id">LVM08008H3G3-M17</param>
-        <param name="lead_mm_per_rev">${lead_mm_per_rev}</param>
-        <param name="lift_sign">${lift_sign}</param>
+        <param name="lead_mm_per_rev">${lift_cfg['lead_mm_per_rev']}</param>
+        <param name="lift_sign">${lift_cfg['lift_sign']}</param>
         <param name="command_units_per_rev">${command_units_per_rev}</param>
         <param name="encoder_counts_per_rev">${encoder_counts_per_rev}</param>
-        <param name="position_min_m">${position_min_m}</param>
-        <param name="position_max_m">${position_max_m}</param>
-        <param name="max_rpm">${max_rpm}</param>
-        <param name="position_limit_recovery_max_rpm">${position_limit_recovery_max_rpm}</param>
+        <param name="position_min_m">${lift_cfg['position_min_m']}</param>
+        <param name="position_max_m">${lift_cfg['position_max_m']}</param>
+        <param name="reset_max_search_travel_m">${lift_cfg['reset_max_search_travel_m']}</param>
+        <param name="max_rpm">${lift_cfg['max_rpm']}</param>
+        <param name="position_limit_recovery_max_rpm">${lift_cfg['position_limit_recovery_max_rpm']}</param>
         <param name="brake_control_enabled">${brake_control_enabled}</param>
         <param name="limit_switch_enabled">${limit_switch_enabled}</param>

File: src/joint_hardware/description/lift_test.urdf.xacro (robot description, xacro)
@@ -15,9 +15,9 @@
   <xacro:arg name="command_units_per_rev" default="10000"/>
   <xacro:arg name="encoder_counts_per_rev" default="131072"/>
-  <xacro:arg name="lead_mm_per_rev" default="10.0"/>
+  <xacro:arg name="lead_mm_per_rev" default="3.333333333"/>
   <xacro:arg name="lift_sign" default="-1.0"/>
   <xacro:arg name="position_min_m" default="-1.0"/>
   <xacro:arg name="position_max_m" default="0.0"/>
-  <xacro:arg name="max_rpm" default="360"/>
+  <xacro:arg name="max_rpm" default="1440"/>
   <xacro:arg name="position_limit_recovery_max_rpm" default="300"/>
   <xacro:arg name="brake_control_enabled" default="false"/>
@@ -36,4 +36,5 @@
   <xacro:arg name="use_persistent_zero_offset" default="false"/>
   <xacro:arg name="zero_offset_file" default="/tmp/joint_hardware_lift_zero_offset.cfg"/>
+  <xacro:property name="lift_cfg" value="${xacro.load_yaml('$(arg hardware_config_file)')}"/>
   <xacro:include filename="$(find joint_hardware)/description/lift.ros2_control.xacro"/>
   <xacro:joint_lift_ros2_control
@@ -79,5 +80,9 @@
     <child link="lift_carriage"/>
     <axis xyz="0 0 1"/>
-    <limit lower="-1.0" upper="0.0" velocity="0.060" effort="1000.0"/>
+    <limit
+      lower="${lift_cfg['position_min_m']}"
+      upper="${lift_cfg['position_max_m']}"
+      velocity="${lift_cfg['max_feedback_velocity_mps']}"
+      effort="1000.0"/>
   </joint>
 </robot>
